Commit message: improve code to work with simulation and added pre-hit placement depending on object

File: object_models/box.urdf (robot description, URDF)
Before this commit: robot simple_box, 1 links, 0 joints
Links:
- link my_box: geometry collision box size=0.23 0.26 0.25; visual box size=0.23 0.26 0.25

File: object_models/table.urdf (robot description, URDF)
Before this commit: robot simple_table, 1 links, 0 joints
Links:
- removed link my_table
- added link table, mass 15; collision box size=0.8 1.6 0.1; visual box size=0.8 1.6 0.1
